File: NaeTime Receiver/NaeTime Receiver.kicad_sch (KiCad schematic)
At the start: 17 parts, among them U15 RX5808_Breakout, U16 RX5808_Breakout, U17 RX5808_Breakout, U18 RX5808_Breakout, U19 RX5808_Breakout, U20 RX5808_Breakout, U21 RX5808_Breakout, U22 RX5808_Breakout

Commit message: Receiver pcb
Parts:
- removed U5: ~, NaeTimeComponentLibrary:RGB LED Header, symbol NaetimeSymbols:LEDHeader
- removed U6: ~, NaeTimeComponentLibrary:DPad Pin Header, symbol NaetimeSymbols:DPad_Pin_Header
- added D1, D2, D3, D4: CLV1L-FKB, NaeTimeComponentLibrary:LED_D5.0mm-4_RGB GBCR, symbol LED:CLV1L-FKB
- added QB1, QG1, QR1: BS170, Package_TO_SOT_THT:TO-92_Inline, symbol Transistor_FET:BS170
- added R1, R10, R4, R7: R2, Resistor_THT:R_Axial_DIN0204_L3.6mm_D1.6mm_P7.62mm_Horizontal, symbol Device:R
- added R11, R2, R5, R8: R3, Resistor_THT:R_Axial_DIN0204_L3.6mm_D1.6mm_P7.62mm_Horizontal, symbol Device:R
- added R12, R3, R6, R9: R4, Resistor_THT:R_Axial_DIN0204_L3.6mm_D1.6mm_P7.62mm_Horizontal, symbol Device:R
- added R13, R14, R15, R16, R17, R18, R19, R20: R1, Resistor_THT:R_Axial_DIN0204_L3.6mm_D1.6mm_P7.62mm_Horizontal, symbol Device:R
- added SW1, SW2, SW3, SW4: SW_Push, Button_Switch_THT:SW_PUSH_6mm_H5mm, symbol Switch:SW_Push
- U15, U16, U17, U18, U19, U20, U21, U22: footprint RX5808_Breakout:RX5808_Breakout -> NaeTimeComponentLibrary:RX5808_Breakout
Connections:
- net +3.3V: no longer U3.8 (3V3)
- net +5V: now also QB1.1 (D), QG1.1 (D), QR1.1 (D)
- net GND: now also LS1.2, D1.1 (A), D2.1 (A), D3.1 (A), D4.1 (A), R13.2, R14.2, R15.2, R16.2, R17.2, R18.2, R19.2, R20.2, SW1.2, SW2.2, SW3.2, SW4.2; no longer LS1.1
- net at U1.8 (25): now also SW1.1
- net at U1.9 (26): now also SW2.1
- net at U1.10 (27): now also SW4.1
- net at U1.11 (14): now also SW3.1
- net at U1.13: now also LS1.1; no longer LS1.2
- net at U1.16 (23/MOSI): now also U3.8 (3V3)
- net RED SWITCH: now reaches U1.17 (22/SCL)
- net RED SWITCH: now also QR1.2 (G)
- net GREEN SWITCH: now reaches U1.6 (32)
- net GREEN SWITCH: now also QG1.2 (G)
- net BLUE SWITCH: now reaches U1.7 (33)
- net BLUE SWITCH: now also QB1.2 (G)
- net at U19.3 (RSSI), U2.2 (19): now also R20.1
- net at U2.6 (16), U22.3 (RSSI): now also R19.1
- net at U16.3 (RSSI), U2.27 (21): now also R15.1
- net at U15.3 (RSSI), U2.26 (20): now also R16.1
- net at U17.3 (RSSI), U2.29 (22): now also R14.1
- net at U18.3 (RSSI), U2.30 (23): now also R13.1
- net at U2.4 (18), U20.3 (RSSI): now also R17.1
- net at U2.5 (17), U21.3 (RSSI): now also R18.1
- new net: D1.4 (BK), R3.2
- new net: D3.3 (GK), R8.2
- new net: D4.2 (RK), R10.2
- new net: D1.2 (RK), R1.2
- new net: D2.2 (RK), R4.2
- new net: D3.2 (RK), R7.2
- new net: D3.4 (BK), R9.2
- new net: D4.3 (GK), R11.2
- new net: D4.4 (BK), R12.2
- new net: D2.3 (GK), R5.2
- new net: D2.4 (BK), R6.2
- new net: D1.3 (GK), R2.2
- new net BLUE: QB1.3 (S), R12.1, R3.1, R6.1, R9.1
- new net GREEN: QG1.3 (S), R11.1, R2.1, R5.1, R8.1
- new net RED: QR1.3 (S), R1.1, R10.1, R4.1, R7.1
